Commit message: [revonic_description] renamed file structure and file paths

File: revonic_description/eva_models/revonic_eva2/revonic_eva2.urdf (robot description, URDF)
Before this commit: robot revonic_eva2, 24 links, 23 joints
Links:
- link base_link: geometry collision mesh filename=package://eva_models/revonic_eva2/meshes/base_link.STL; visual mesh filename=package://eva_models/revonic_eva2/meshes/base_link.STL
- link crab_steer_assy1: geometry collision mesh filename=package://eva_models/revonic_eva2/meshes/crab_steer_assy1.S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; visual mesh filename=package://eva_models/revonic_eva2/meshes/crab_steer_assy1.S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
- link crab_steer_assy2: geometry collision mesh filename=package://eva_models/revonic_eva2/meshes/crab_steer_assy2.S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; visual mesh filename=package://eva_models/revonic_eva2/meshes/crab_steer_assy2.S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
- link crab_steer_assy3: geometry collision mesh filename=package://eva_models/revonic_eva2/meshes/crab_steer_assy3.S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; visual mesh filename=package://eva_models/revonic_eva2/meshes/crab_steer_assy3.S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
- link crab_steer_assy4: geometry collision mesh filename=package://eva_models/revonic_eva2/meshes/crab_steer_assy4.S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; visual mesh filename=package://eva_models/revonic_eva2/meshes/crab_steer_assy4.S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
- link differential_bar: geometry collision mesh filename=package://eva_models/revonic_eva2/meshes/differential_bar.S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; visual mesh filename=package://eva_models/revonic_eva2/meshes/differential_bar.S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
- link differential_connection_rodend1: geometry collision mesh filename=package://eva_models/revonic_eva2/meshes/differential_conne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; visual mesh filename=package://eva_models/revonic_eva2/meshes/differential_conne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
- link differential_connection_rodend2: geometry collision mesh filename=package://eva_models/revonic_eva2/meshes/differential_conne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; visual mesh filename=package://eva_models/revonic_eva2/meshes/differential_conne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
- link differential_connection_rodend3: geometry collision mesh filename=package://eva_models/revonic_eva2/meshes/differential_conne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; visual mesh filename=package://eva_models/revonic_eva2/meshes/differential_conne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
- link differential_connection_rodend4: geometry collision mesh filename=package://eva_models/revonic_eva2/meshes/differential_conne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; visual mesh filename=package://eva_models/revonic_eva2/meshes/differential_conne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
- link differential_connection_virt1_rodend1: geometry collision mesh filename=package://eva_models/revonic_eva2/meshes/differential_conne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; visual mesh filename=package://eva_models/revonic_eva2/meshes/differential_conne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
- link differential_connection_virt1_rodend2: geometry collision mesh filename=package://eva_models/revonic_eva2/meshes/differential_conne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; visual mesh filename=package://eva_models/revonic_eva2/meshes/differential_conne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
- link differential_connection_virt1_rodend3: geometry collision mesh filename=package://eva_models/revonic_eva2/meshes/differential_conne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; visual mesh filename=package://eva_models/revonic_eva2/meshes/differential_conne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
- link differential_connection_virt1_rodend4: geometry collision mesh filename=package://eva_models/revonic_eva2/meshes/differential_conne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; visual mesh filename=package://eva_models/revonic_eva2/meshes/differential_conne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
- link differential_connection_virt2_rodend1: geometry collision mesh filename=package://eva_models/revonic_eva2/meshes/differential_conne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; visual mesh filename=package://eva_models/revonic_eva2/meshes/differential_conne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
- link differential_connection_virt2_rodend2: geometry collision mesh filename=package://eva_models/revonic_eva2/meshes/differential_conne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; visual mesh filename=package://eva_models/revonic_eva2/meshes/differential_conne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
- link differential_connection_virt2_rodend3: geometry collision mesh filename=package://eva_models/revonic_eva2/meshes/differential_conne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; visual mesh filename=package://eva_models/revonic_eva2/meshes/differential_conne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
- link differential_connection_virt2_rodend4: geometry collision mesh filename=package://eva_models/revonic_eva2/meshes/differential_conne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; visual mesh filename=package://eva_models/revonic_eva2/meshes/differential_conne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
- link drive_hex_wheel1: geometry collision mesh filename=package://eva_models/revonic_eva2/meshes/drive_hex_wheel1.S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; visual mesh filename=package://eva_models/revonic_eva2/meshes/drive_hex_wheel1.S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
- link drive_hex_wheel2: geometry collision mesh filename=package://eva_models/revonic_eva2/meshes/drive_hex_wheel2.S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; visual mesh filename=package://eva_models/revonic_eva2/meshes/drive_hex_wheel2.S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
- link drive_hex_wheel3: geometry collision mesh filename=package://eva_models/revonic_eva2/meshes/drive_hex_wheel3.S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; visual mesh filename=package://eva_models/revonic_eva2/meshes/drive_hex_wheel3.S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
- link drive_hex_wheel4: geometry collision mesh filename=package://eva_models/revonic_eva2/meshes/drive_hex_wheel4.S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; visual mesh filename=package://eva_models/revonic_eva2/meshes/drive_hex_wheel4.S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
- link suspension_arm1: geometry collision mesh filename=package://eva_models/revonic_eva2/meshes/suspension_arm1.STL; visual mesh filename=package://eva_models/revonic_eva2/meshes/suspension_arm1.STL
- link suspension_arm2: geometry collision mesh filename=package://eva_models/revonic_eva2/meshes/suspension_arm2.STL; visual mesh filename=package://eva_models/revonic_eva2/meshes/suspension_arm2.STL

Commit message: [revonic_description] fixed path errors and added continuous joints

File: revonic_description/eva_models/revonic_eva2/revonic_eva2.urdf (robot description, URDF)
Before this commit: robot revonic_eva2, 24 links, 23 joints
Links:
- added link kdl_dummy_root
- link base_link: geometry collision mesh filename=package://revonic_description/eva_models/revonic_eva2/meshe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; visual mesh filename=package://revonic_description/eva_models/revonic_eva2/meshe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
- link crab_steer_assy1: geometry collision mesh filename=package://revonic_description/eva_models/revonic_eva2/meshe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; visual mesh filename=package://revonic_description/eva_models/revonic_eva2/meshe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
- link crab_steer_assy2: geometry collision mesh filename=package://revonic_description/eva_models/revonic_eva2/meshe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; visual mesh filename=package://revonic_description/eva_models/revonic_eva2/meshe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
- link crab_steer_assy3: geometry collision mesh filename=package://revonic_description/eva_models/revonic_eva2/meshe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; visual mesh filename=package://revonic_description/eva_models/revonic_eva2/meshe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
- link crab_steer_assy4: geometry collision mesh filename=package://revonic_description/eva_models/revonic_eva2/meshe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; visual mesh filename=package://revonic_description/eva_models/revonic_eva2/meshe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
- link differential_bar: geometry collision mesh filename=package://revonic_description/eva_models/revonic_eva2/meshe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; visual mesh filename=package://revonic_description/eva_models/revonic_eva2/meshe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
- link differential_connection_rodend1: geometry collision mesh filename=package://revonic_description/eva_models/revonic_eva2/meshe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; visual mesh filename=package://revonic_description/eva_models/revonic_eva2/meshe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
- link differential_connection_rodend2: geometry collision mesh filename=package://revonic_description/eva_models/revonic_eva2/meshe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; visual mesh filename=package://revonic_description/eva_models/revonic_eva2/meshe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
- link differential_connection_rodend3: geometry collision mesh filename=package://revonic_description/eva_models/revonic_eva2/meshe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; visual mesh filename=package://revonic_description/eva_models/revonic_eva2/meshe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
- link differential_connection_rodend4: geometry collision mesh filename=package://revonic_description/eva_models/revonic_eva2/meshe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; visual mesh filename=package://revonic_description/eva_models/revonic_eva2/meshe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
- link differential_connection_virt1_rodend1: geometry collision mesh filename=package://revonic_description/eva_models/revonic_eva2/meshe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; visual mesh filename=package://revonic_description/eva_models/revonic_eva2/meshe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
- link differential_connection_virt1_rodend2: geometry collision mesh filename=package://revonic_description/eva_models/revonic_eva2/meshe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; visual mesh filename=package://revonic_description/eva_models/revonic_eva2/meshe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
- link differential_connection_virt1_rodend3: geometry collision mesh filename=package://revonic_description/eva_models/revonic_eva2/meshe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; visual mesh filename=package://revonic_description/eva_models/revonic_eva2/meshe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
- link differential_connection_virt1_rodend4: geometry collision mesh filename=package://revonic_description/eva_models/revonic_eva2/meshe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; visual mesh filename=package://revonic_description/eva_models/revonic_eva2/meshe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
- link differential_connection_virt2_rodend1: geometry collision mesh filename=package://revonic_description/eva_models/revonic_eva2/meshe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; visual mesh filename=package://revonic_description/eva_models/revonic_eva2/meshe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
- link differential_connection_virt2_rodend2: geometry collision mesh filename=package://revonic_description/eva_models/revonic_eva2/meshe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; visual mesh filename=package://revonic_description/eva_models/revonic_eva2/meshe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
- link differential_connection_virt2_rodend3: geometry collision mesh filename=package://revonic_description/eva_models/revonic_eva2/meshe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; visual mesh filename=package://revonic_description/eva_models/revonic_eva2/meshe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
- link differential_connection_virt2_rodend4: geometry collision mesh filename=package://revonic_description/eva_models/revonic_eva2/meshe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; visual mesh filename=package://revonic_description/eva_models/revonic_eva2/meshe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
- link drive_hex_wheel1: geometry collision mesh filename=package://revonic_description/eva_models/revonic_eva2/meshe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; visual mesh filename=package://revonic_description/eva_models/revonic_eva2/meshe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
- link drive_hex_wheel2: geometry collision mesh filename=package://revonic_description/eva_models/revonic_eva2/meshe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; visual mesh filename=package://revonic_description/eva_models/revonic_eva2/meshe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
- link drive_hex_wheel3: geometry collision mesh filename=package://revonic_description/eva_models/revonic_eva2/meshe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; visual mesh filename=package://revonic_description/eva_models/revonic_eva2/meshe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
- link drive_hex_wheel4: geometry collision mesh filename=package://revonic_description/eva_models/revonic_eva2/meshe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; visual mesh filename=package://revonic_description/eva_models/revonic_eva2/meshe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
- link suspension_arm1: geometry collision mesh filename=package://revonic_description/eva_models/revonic_eva2/meshe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; visual mesh filename=package://revonic_description/eva_models/revonic_eva2/meshe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
- link suspension_arm2: geometry collision mesh filename=package://revonic_description/eva_models/revonic_eva2/meshe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; visual mesh filename=package://revonic_description/eva_models/revonic_eva2/meshe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
Joints:
- added joint kdl_dummy_root_joint: type fixed, parent kdl_dummy_root, child base_link, origin xyz=0 0 0.1325 rpy=0 0 0
- joint drive_act_joint1: type revolute -> continuous
- joint drive_act_joint2: type revolute -> continuous
- joint drive_act_joint3: type revolute -> continuous
- joint drive_act_joint4: type revolute -> continuous

Commit message: [revonic_description] Defined virtual ball joints for differential

File: revonic_description/eva_models/revonic_eva2/revonic_eva2.urdf (robot description, URDF)
Before this commit: robot revonic_eva2, 25 links, 24 joints
Links:
- link differential_connection_virt1_rodend1: geometry 
- link differential_connection_virt1_rodend2: geometry 
- link differential_connection_virt1_rodend3: geometry 
- link differential_connection_virt1_rodend4: geometry 
- link differential_connection_virt2_rodend1: geometry 
- link differential_connection_virt2_rodend2: geometry 
- link differential_connection_virt2_rodend3: geometry 
- link differential_connection_virt2_rodend4: geometry 

Commit message: [revonic_description] Modified ball-joint relations and axes of rotation

File: revonic_description/eva_models/revonic_eva2/revonic_eva2.urdf (robot description, URDF)
Before this commit: robot revonic_eva2, 25 links, 24 joints
Joints:
- joint differential_connection1_joint2: axis -1 0 0 -> 0 -1 0
- joint differential_connection2_joint1: axis 0 1 0 -> 0 0 -1
- joint differential_connection2_joint2: axis -1 0 0 -> 0 -1 0
- joint differential_connection2_joint3: origin xyz=0 0 0 rpy=0 0 0 -> xyz=-0.00014998 0.0021259 -0.098347 rpy=0 0 0; parent differential_connection_virt2_rodend2 -> differential_connection_rodend1
- joint differential_connection3_joint2: axis -1 0 0 -> 0 -1 0
- joint differential_connection4_joint1: axis 0 1 0 -> -1 0 0
- joint differential_connection4_joint2: axis -1 0 0 -> 0 -1 0
- joint differential_connection4_joint3: origin xyz=0 0 0 rpy=0 0 0 -> xyz=-0.00014998 -0.0021259 -0.098347 rpy=0 0 0; parent differential_connection_virt2_rodend4 -> differential_connection_rodend3
